File: EDA/EDA.kicad_pcb (KiCad board)
At the start: 2 copper layers, 85 x 52.8 mm, 34 parts, among them J1 ENCODER - AMT 10, J2 USB_A, J3 H Bridges, U1 ATtiny414-SS, U2 A4950E, U3 TPS61040DRV, U4 CH340N, U5 LSF0204, U6 TVS1400DRV, U7 TPS62140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

Commit message: t
Parts:
- moved U8 91.3 mm to (193.2, 101.2)
- moved C10 85.7 mm to (187.4, 114.0), turned to -90 degrees
- moved R7 83.8 mm to (190.8, 118.2), turned to 180 degrees
- moved C9 83.3 mm to (184.8, 114.0), turned to 90 degrees
- moved C7 82.4 mm to (179.1, 120.5)
- moved C11 79.8 mm to (182.1, 114.1), turned to 90 degrees
- moved D2 77.8 mm to (176.1, 112.9), turned to 90 degrees
- moved R5 73.9 mm to (175.3, 121.3), turned to -90 degrees
- moved C8 73.4 mm to (175.4, 108.4), turned to -90 degrees
- moved R6 70.5 mm to (175.3, 117.2)
- moved U7 69.4 mm to (153.1, 107.7)
- moved R1 66.6 mm to (176.1, 79.5), turned to 180 degrees
- moved C1 62.9 mm to (168.3, 82.7)
- moved L1 62.7 mm to (159.2, 112.9)
- moved U3 62.1 mm to (172.3, 108.3)
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Routing:
- net +5V: track 0.00 -> 106.0 mm, vias 0 -> 6
- net +3V3: track 0.00 -> 99.2 mm, vias 0 -> 8
- net /3V3_ENC_A: track 0.00 -> 38.8 mm, vias 0 -> 2
- net /UPDI: track 0.00 -> 37.2 mm
- net /3V3_ENC_B: track 0.00 -> 35.6 mm
- net VBAT: track 0.00 -> 34.9 mm
- net Net-(J2-D+): track 0.00 -> 31.4 mm, vias 0 -> 2
- net /5V_ENC_A: track 0.00 -> 28.5 mm
- net /5V_ENC_B: track 0.00 -> 28.1 mm
- net Net-(J2-D-): track 0.00 -> 27.1 mm, vias 0 -> 2
- net /VBB: track 0.00 -> 26.8 mm
- net /H Bridge 2: track 0.00 -> 26.4 mm
- net /H Bridge 1: track 0.00 -> 24.3 mm
- net Net-(J3-Pin_1): track 0.00 -> 22.1 mm
- net Net-(J3-Pin_2): track 0.00 -> 19.3 mm
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
Commit message: zone
Routing:
- added copper zone on F.Cu, net GND
Changed lines of the file:
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@@
 		(net 35)
 	)
+	(zone
+		(net 2)
+		(net_name "GND")
+		(layer "F.Cu")
+		(hatch edge 0.5)
+		(connect_pads
+			(clearance 0.5)
+		)
+		(min_thickness 0.25)
+		(filled_areas_thickness no)
+		(fill yes
+			(thermal_gap 0.5)
+			(thermal_bridge_width 0.5)
+			(island_removal_mode 1)
+			(island_area_min 10)
+		)
+		(polygon
+			(pts
+				(xy 221.6 125.7) (xy 221.6 71.8) (xy 130.7 71.2) (xy 135.7 127.7)
+			)
+		)
+	)
 )

Commit message: t
Connections:
- U3 pad 6: unconnected-(U3-SW-Pad6) -> Net-(D2-A)
Routing:
- net +5V: track 106.0 -> 113.2 mm
- net Net-(U7-SS/TR): track 0.00 -> 4.22 mm
Changed lines of the file:
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@@
 	(net 34 "unconnected-(U1-PB0-Pad9)")
 	(net 35 "/3V3_ENC_A")
-	(net 36 "unconnected-(U3-SW-Pad6)")
-	(net 37 "unconnected-(U3-EN-Pad3)")
-	(net 38 "unconnected-(U3-NC-Pad5)")
-	(net 39 "unconnected-(U4-~{RTS}-Pad4)")
-	(net 40 "unconnected-(U5-B3-Pad11)")
-	(net 41 "unconnected-(U5-A3-Pad4)")
-	(net 42 "unconnected-(U5-A4-Pad5)")
-	(net 43 "unconnected-(U5-B4-Pad10)")
+	(net 36 "unconnected-(U3-EN-Pad3)")
+	(net 37 "unconnected-(U3-NC-Pad5)")
+	(net 38 "unconnected-(U4-~{RTS}-Pad4)")
+	(net 39 "unconnected-(U5-B3-Pad11)")
+	(net 40 "unconnected-(U5-A3-Pad4)")
+	(net 41 "unconnected-(U5-A4-Pad5)")
+	(net 42 "unconnected-(U5-B4-Pad10)")
 	(footprint "Inductor_SMD:L_Vishay_IHLP-1212"
 		(layer "F.Cu")
@@
 			(layers "F.Cu" "F.Paste" "F.Mask")
 			(roundrect_rratio 0.25)
-			(net 39 "unconnected-(U4-~{RTS}-Pad4)")
+			(net 38 "unconnected-(U4-~{RTS}-Pad4)")
 			(pinfunction "~{RTS}")
 			(pintype "output+no_connect")
@@
 			(size 0.28 0.85)
 			(layers "F.Cu" "F.Paste" "F.Mask")
-			(net 41 "unconnected-(U5-A3-Pad4)")
+			(net 40 "unconnected-(U5-A3-Pad4)")
 			(pinfunction "A3")
 			(pintype "bidirectional+no_connect")
@@
 			(size 0.28 0.85)
 			(layers "F.Cu" "F.Paste" "F.Mask")
-			(net 42 "unconnected-(U5-A4-Pad5)")
+			(net 41 "unconnected-(U5-A4-Pad5)")
 			(pinfunction "A4")
 			(pintype "bidirectional+no_connect")
@@
 			(size 0.28 0.85)
 			(layers "F.Cu" "F.Paste" "F.Mask")
-			(net 43 "unconnected-(U5-B4-Pad10)")
+			(net 42 "unconnected-(U5-B4-Pad10)")
 			(pinfunction "B4")
 			(pintype "bidirectional+no_connect")
@@
 			(size 0.28 0.85)
 			(layers "F.Cu" "F.Paste" "F.Mask")
-			(net 40 "unconnected-(U5-B3-Pad11)")
+			(net 39 "unconnected-(U5-B3-Pad11)")
 			(pinfunction "B3")
 			(pintype "bidirectional+no_connect")
@@
 			(layers "F.Cu" "F.Paste" "F.Mask")
 			(roundrect_rratio 0.25)
-			(net 37 "unconnected-(U3-EN-Pad3)")
+			(net 36 "unconnected-(U3-EN-Pad3)")
 			(pinfunction "EN")
 			(pintype "input")
@@
 			(layers "F.Cu" "F.Paste" "F.Mask")
 			(roundrect_rratio 0.25)
-			(net 38 "unconnected-(U3-NC-Pad5)")
+			(net 37 "unconnected-(U3-NC-Pad5)")
 			(pinfunction "NC")
 			(pintype "no_connect")
@@
 			(layers "F.Cu" "F.Paste" "F.Mask")
 			(roundrect_rratio 0.25)
-			(net 36 "unconnected-(U3-SW-Pad6)")
+			(net 10 "Net-(D2-A)")
 			(pinfunction "SW")
 			(pintype "power_out")
@@
 	)
 	(segment
+		(start 158.325 109.6)
+		(end 155.8 109.6)
+		(width 0.2)
+		(layer "F.Cu")
+		(net 6)
+	)
+	(segment
+		(start 155.8 109.6)
+		(end 154.6 108.4)
+		(width 0.2)
+		(layer "F.Cu")
+		(net 6)
+	)
+	(segment
 		(start 161.115 109.975)
 		(end 161.115 109.3)
@@
 	)
 	(segment
+		(start 156.701659 107.865)
+		(end 153.324876 104.488217)
+		(width 0.2)
+		(layer "F.Cu")
+		(net 7)
+	)
+	(segment
 		(start 161 109.3)
 		(end 159.565 107.865)
@@
 		(width 0.2)
 		(layer "F.Cu")
+		(net 7)
+	)
+	(segment
+		(start 159.19 107.865)
+		(end 156.701659 107.865)
+		(width 0.2)
+		(layer "F.Cu")
