File: EDA/EDA.kicad_sch (KiCad schematic)
At the start: 34 parts, among them J1 ENCODER - AMT 10, J2 USB_A, J3 H Bridges, U1 ATtiny414-SS, U2 A4950E, U3 TPS61040DRV, U4 CH340N, U5 LSF0204, U6 TVS1400DRV, U7 TPS62140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

Commit message: t
Connections:
- net at U3.6 (SW): now also D2.2 (A), L2.2
Changed lines of the file:
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@@
+	)
+	(junction
+		(at 171.45 133.35)
+		(diameter 0)
+		(color 0 0 0 0)
 	)
 	(junction
@@
 	(wire
 		(pts
-			(xy 167.64 133.35) (xy 173.99 133.35)
+			(xy 167.64 133.35) (xy 171.45 133.35)
 		)
 		(stroke
@@
 	(wire
 		(pts
+			(xy 171.45 133.35) (xy 171.45 142.24)
+		)
+		(stroke
+			(width 0)
+			(type default)
+		)
+	)
+	(wire
+		(pts
 			(xy 38.1 62.23) (xy 62.23 62.23)
 		)
@@
 		(pts
 			(xy 36.83 48.26) (xy 52.07 48.26)
+		)
+		(stroke
+			(width 0)
+			(type default)
+		)
+	)
+	(wire
+		(pts
+			(xy 171.45 133.35) (xy 173.99 133.35)
 		)
 		(stroke
@@
 	)
 	(label "H Bridge 1"
-		(at 127 116.84 180)
+		(at 127 116.84 0)
 		(effects
 			(font
 				(size 1.27 1.27)
 			)
-			(justify right bottom)
-		)
-	)
+			(justify left bottom)
+		)
+	)
